File: audio_and_microphone/audio_and_microphone.kicad_sch (KiCad schematic)
At the start: 33 parts, among them J1 Conn_01x02, J10 Conn_01x03_Socket, J11 Conn_01x02, J2 Conn_01x02, J3 Conn_01x02, J4 Conn_01x02, J5 Conn_01x10_MountingPin, J6 Conn_01x08_MountingPin, J7 Conn_01x08_MountingPin, J8 Conn_01x06_MountingPin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

Commit message: updated and imported footprints to match altium
Parts:
- C1, C14, C19, C2, C26, C27, C3, C4, C5: footprint Capacitor_SMD:C_0201_0603Metric -> C1608X5R1E105K080AC:CAPC1608X90N
- R1, R18, R19, R2, R3, R32, R36, R4, R5: footprint Resistor_SMD:R_0201_0603Metric -> RC0603FR_072KL:R0603
Changed lines of the file:
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@@
 			)
 		)
-		(property "Footprint" "Capacitor_SMD:C_0201_0603Metric"
+		(property "Footprint" "C1608X5R1E105K080AC:CAPC1608X90N"
 			(at 119.38 169.2148 0)
 			(effects
@@
 			)
 		)
-		(property "Footprint" "Resistor_SMD:R_0201_0603Metric"
+		(property "Footprint" "RC0603FR_072KL:R0603"
 			(at 129.286 106.934 90)
 			(effects
@@
 			)
 		)
-		(property "Footprint" "Capacitor_SMD:C_0201_0603Metric"
+		(property "Footprint" "C1608X5R1E105K080AC:CAPC1608X90N"
 			(at 54.3052 105.41 0)
 			(effects
@@
 			)
 		)
-		(property "Footprint" "Capacitor_SMD:C_0201_0603Metric"
+		(property "Footprint" "C1608X5R1E105K080AC:CAPC1608X90N"
 			(at 132.08 169.2148 0)
 			(effects
@@
 			)
 		)
-		(property "Footprint" "Capacitor_SMD:C_0201_0603Metric"
+		(property "Footprint" "C1608X5R1E105K080AC:CAPC1608X90N"
 			(at 212.09 107.95 0)
 			(effects
@@
 			)
 		)
-		(property "Footprint" "Capacitor_SMD:C_0201_0603Metric"
+		(property "Footprint" "C1608X5R1E105K080AC:CAPC1608X90N"
 			(at 47.9552 105.41 0)
 			(effects
@@
 			)
 		)
-		(property "Footprint" "Resistor_SMD:R_0201_0603Metric"
+		(property "Footprint" "RC0603FR_072KL:R0603"
 			(at 188.976 150.114 90)
 			(effects
@@
 			)
 		)
-		(property "Footprint" "Capacitor_SMD:C_0201_0603Metric"
+		(property "Footprint" "C1608X5R1E105K080AC:CAPC1608X90N"
 			(at 76.2 129.54 0)
 			(effects
@@
 			)
 		)
-		(property "Footprint" "Resistor_SMD:R_0201_0603Metric"
+		(property "Footprint" "RC0603FR_072KL:R0603"
 			(at 114.554 141.224 90)
 			(effects
@@
 			)
 		)
-		(property "Footprint" "Capacitor_SMD:C_0201_0603Metric"
+		(property "Footprint" "C1608X5R1E105K080AC:CAPC1608X90N"
 			(at 124.1552 153.67 0)
 			(effects
@@
 			)
 		)
-		(property "Footprint" "Capacitor_SMD:C_0201_0603Metric"
+		(property "Footprint" "C1608X5R1E105K080AC:CAPC1608X90N"
 			(at 116.84 99.3648 0)
 			(effects
@@
 			)
 		)
-		(property "Footprint" "Resistor_SMD:R_0201_0603Metric"
+		(property "Footprint" "RC0603FR_072KL:R0603"
 			(at 208.026 144.526 90)
 			(effects
@@
 			)
 		)
-		(property "Footprint" "Resistor_SMD:R_0201_0603Metric"
+		(property "Footprint" "RC0603FR_072KL:R0603"
 			(at 114.554 78.994 90)
 			(effects
@@
 			)
 		)
-		(property "Footprint" "Resistor_SMD:R_0201_0603Metric"
+		(property "Footprint" "RC0603FR_072KL:R0603"
 			(at 55.626 121.666 90)
 			(effects
@@
 			)
 		)
-		(property "Footprint" "Resistor_SMD:R_0201_0603Metric"
+		(property "Footprint" "RC0603FR_072KL:R0603"
 			(at 67.056 124.206 90)
 			(effects
@@
 			)
 		)
-		(property "Footprint" "Resistor_SMD:R_0201_0603Metric"
+		(property "Footprint" "RC0603FR_072KL:R0603"
 			(at 133.604 141.224 90)
 			(effects
@@
 			)
 		)
-		(property "Footprint" "Resistor_SMD:R_0201_0603Metric"
+		(property "Footprint" "RC0603FR_072KL:R0603"
 			(at 122.936 176.784 90)
 			(effects
@@
 			)
 		)
-		(property "Footprint" "Capacitor_SMD:C_0201_0603Metric"
+		(property "Footprint" "C1608X5R1E105K080AC:CAPC1608X90N"
 			(at 131.7752 90.17 0)
 			(effects

Commit message: fixed ground island in pcb
Connections:
- net +3V3: now also J7.1 (Pin_1), J7.2 (Pin_2), J7.4 (Pin_4)
- net GND: now also J7.6 (Pin_6), J7.7 (Pin_7)
- no-connect marks 0 -> 62
Other:
- moved on the sheet: J7
