File: audio_and_microphone/audio_and_microphone.kicad_sch (KiCad schematic)
At the start: 32 parts, among them J1 Conn_01x08_MountingPin, J10 Conn_01x02_Pin, J2 Conn_01x03_MountingPin, J3 Conn_01x06_MountingPin, J4 Conn_01x03_Pin, J5 Conn_01x02, J6 Conn_01x10_MountingPin, J7 Conn_01x02, J8 Conn_01x02, J9 Conn_01x02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

Commit message: updated pcb with two sides and back side with voltage
Parts:
- removed R2, R4: 22k, Resistor_SMD:R_0603_1608Metric_Pad0.98x0.95mm_HandSolder, symbol Device:R_US
- R1, R3: value 4.7k -> 26.7k
Connections:
- net at C3.2, J8.2 (Pin_2): now also R3.2
- net at R1.2: now also C1.1, R3.1
Changed lines of the file:
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@@
 	(wire
 		(pts
-			(xy 144.78 119.38) (xy 146.05 119.38)
+			(xy 116.84 119.38) (xy 127 119.38)
 		)
 		(stroke
@@
 	(wire
 		(pts
+			(xy 137.16 119.38) (xy 146.05 119.38)
+		)
+		(stroke
+			(width 0)
+			(type default)
+		)
+	)
+	(wire
+		(pts
 			(xy 52.07 110.49) (xy 59.69 110.49)
 		)
@@
 	(wire
 		(pts
-			(xy 124.46 119.38) (xy 127 119.38)
-		)
-		(stroke
-			(width 0)
-			(type default)
-		)
-	)
-	(wire
-		(pts
 			(xy 50.8 82.55) (xy 50.8 87.63)
 		)
@@
 			)
 		)
-		(property "Value" "4.7k"
+		(property "Value" "26.7k"
 			(at 113.03 115.57 90)
 			(effects
@@
 	)
 	(symbol
-		(lib_id "Device:R_US")
-		(at 120.65 119.38 90)
-		(unit 1)
-		(exclude_from_sim no)
-		(in_bom yes)
-		(on_board yes)
-		(dnp no)
-		(fields_autoplaced yes)
-		(property "Reference" "R2"
-			(at 120.65 113.03 90)
-			(effects
-				(font
-					(size 1.27 1.27)
-				)
-			)
-		)
-		(property "Value" "22k"
-			(at 120.65 115.57 90)
-			(effects
-				(font
-					(size 1.27 1.27)
-				)
-			)
-		)
-		(property "Footprint" "Resistor_SMD:R_0603_1608Metric_Pad0.98x0.95mm_HandSolder"
-			(at 120.904 118.364 90)
-			(effects
-				(font
-					(size 1.27 1.27)
-				)
-				(hide yes)
-			)
-		)
-		(property "Datasheet" "~"
-			(at 120.65 119.38 0)
-			(effects
-				(font
-					(size 1.27 1.27)
-				)
-				(hide yes)
-			)
-		)
-		(property "Description" "Resistor, US symbol"
-			(at 120.65 119.38 0)
-			(effects
-				(font
-					(size 1.27 1.27)
-				)
-				(hide yes)
-			)
-		)
-		(pin "2"
-		)
-		(pin "1"
-		)
-		(instances
-			(project "audio_and_microphone"
-				(path "/6041ce46-c287-4741-ac80-b7b1d4df1348"
-					(reference "R2")
-					(unit 1)
-				)
-			)
-		)
-	)
-	(symbol
 		(lib_id "Device:C")
 		(at 50.8 91.44 0)
@@
 			)
 		)
-		(property "Value" "4.7k"
+		(property "Value" "26.7k"
 			(at 133.35 115.57 90)
 			(effects
@@
 					(unit 1)
 				)
-			)
-		)
-	)
-	(symbol
-		(lib_id "Device:R_US")
-		(at 140.97 119.38 90)
-		(unit 1)
-		(exclude_from_sim no)
-		(in_bom yes)
-		(on_board yes)
-		(dnp no)
-		(property "Reference" "R4"
-			(at 140.97 113.03 90)
-			(effects
-				(font
-					(size 1.27 1.27)
-				)
-			)
-		)
-		(property "Value" "22k"
-			(at 140.97 115.57 90)
-			(effects
-				(font
-					(size 1.27 1.27)
-				)
-			)
-		)
-		(property "Footprint" "Resistor_SMD:R_0603_1608Metric_Pad0.98x0.95mm_HandSolder"
-			(at 141.224 118.364 90)
-			(effects
-				(font
-					(size 1.27 1.27)
-				)
-				(hide yes)
-			)
-		)
-		(property "Datasheet" "~"
-			(at 140.97 119.38 0)
-			(effects
-				(font
-					(size 1.27 1.27)
-				)
-				(hide yes)
-			)
-		)
-		(property "Description" "Resistor, US symbol"
-			(at 140.97 119.38 0)
-			(effects
-				(font
-					(size 1.27 1.27)
-				)
-				(hide yes)
-			)
-		)
-		(pin "2"
-		)
-		(pin "1"
-		)
-		(instances
-			(project "audio_and_microphone"
-				(path "/6041ce46-c287-4741-ac80-b7b1d4df1348"
-					(reference "R4")
-					(unit 1)
-				)
