File: 065-0200_Main Board (Rev E)/065-0200_Page 2 Power.kicad_sch (KiCad schematic)
At the start: 65 parts, among them J1 UJ32-C-H-G-H2-SMT-TR, J3 ${PART NUMBER}, Q1 ${PART NUMBER}, SW1 ${PART NUMBER}, U14 ${PART NUMBER}, U15 ${PART NUMBER}

Commit message: Fix Altium import template variables and footprints in Rev E schematics
- Replace 52 ${PART NUMBER} template variables with actual part numbers
- Replace 180 Altium footprint references with KiCad standard library equivalents
- Placeholders set for BM833, 2SMPP03, custom connectors (need manual assignment)

Co-Authored-By: Claude Sonnet 4.6 <noreply@anthropic.com>
Parts:
- C1, C10, C2, C31, C36, C37, C44, C9: footprint Discretes.PcbLib:CAP_0603 -> Capacitor_SMD:C_0603_1608Metric
- C30, C33, C34: value ${PART NUMBER} -> CL10A226MO7JZNC; footprint Discretes.PcbLib:CAP_0603 -> Capacitor_SMD:C_0603_1608Metric
- C35: value ${PART NUMBER} -> C0603C102K5RACTU; footprint Discretes.PcbLib:CAP_0603 -> Capacitor_SMD:C_0603_1608Metric
- D1: footprint Discretes.PcbLib:SOD-123_BD -> Diode_SMD:D_SOD-123
- D12, D7: value ${PART NUMBER} -> APT1608ZGCK; footprint Discretes.PcbLib:LED_0603 -> LED_SMD:LED_0603_1608Metric
- D2, D3: value ${PART NUMBER} -> D5V0H1B2LP-7B; footprint DFN2_1.01X0.61_0.65P -> Diode_SMD:D_DFN-2_1x0.6mm_P0.65mm
- F1: value ${PART NUMBER} -> C2Q 2.5; footprint Discretes.PcbLib:RES_0603 -> Resistor_SMD:R_0603_1608Metric
- FD1, FD2, FD3, FD4, FD5, FD6: value ${PART NUMBER} -> DNI; footprint Fiducial_30 -> Fiducial:Fiducial_1mm_Silk
- J1: footprint CUI_UJ32-C-H-G-H2-SMT-TR -> Connector_USB:USB_C_Receptacle_HRO_TYPE-C-31-M-12
- J3: value ${PART NUMBER} -> 0022035025; footprint Molex_2P-2.50_22035025 -> Connector_PinHeader_2.54mm:PinHeader_1x02_P2.54mm_Vertical
- L1: value ${PART NUMBER} -> CIGT252012LMR47MNE; footprint L_1008 -> Inductor_SMD:L_1008_2520Metric
- MH1, MH4, MH7, MH8: value ${PART NUMBER} -> DNI; footprint MH_M3_Pad -> MountingHole:MountingHole_3.2mm_M3_Pad
- MH10, MH11, MH2, MH3, MH5, MH6, MH9: value ${PART NUMBER} -> DNI; footprint MH_M2.5_Pad -> MountingHole:MountingHole_2.7mm_M2.5_Pad
- Q1: value ${PART NUMBER} -> CSD25402Q3A; footprint Q_8VSON_PCH _NOVIA -> Package_DFN_QFN:VSON-8-1EP_2x2mm_P0.5mm_EP0.9x1.7mm
- R1, R2, R3, R40, R41, R45, R46, R47, R48, R49, R51, R52, R54, R55, R56, R69, R7: footprint Discretes.PcbLib:RES_0603 -> Resistor_SMD:R_0603_1608Metric
- R42, R50, R8: footprint Discretes.PcbLib:RES_0805 -> Resistor_SMD:R_0805_2012Metric
- SW1: value ${PART NUMBER} -> 3-1437565-0; footprint SW_TE_3-1437565-0 -> Button_Switch_SMD:SW_TE_3-1437565-0
- TP1, TP2, TP7: footprint Connectors.PcbLib:TP_SMT_0.030 -> TestPoint:TestPoint_Pad_D0.8mm
- U14: value ${PART NUMBER} -> TPS63802DLAT; footprint TI-VSON-HR-10 -> Package_DFN_QFN:VSON-10-1EP_3x3mm_P0.5mm_EP1.7x1.7mm
- U15: value ${PART NUMBER} -> NPM1300-QEAA-R; footprint QFN-32_5X5_EXP -> Package_DFN_QFN:QFN-32-1EP_5x5mm_P0.5mm_EP3.1x3.1mm

Commit message: Fix footprint names to match installed KiCad library
Correct 30 footprint references where library name or footprint name
didn't match KiCad's actual installed libraries (Package_SON vs
Package_DFN_QFN, SOT-363_SC-70-6, Fiducial, SOT-883, etc.)

Co-Authored-By: Claude Sonnet 4.6 <noreply@anthropic.com>
Parts:
- D2, D3: footprint Diode_SMD:D_DFN-2_1x0.6mm_P0.65mm -> Package_TO_SOT_SMD:SOT-883
- FD1, FD2, FD3, FD4, FD5, FD6: footprint Fiducial:Fiducial_1mm_Silk -> Fiducial:Fiducial_1mm_Mask2mm
- Q1: footprint Package_DFN_QFN:VSON-8-1EP_2x2mm_P0.5mm_EP0.9x1.7mm -> Package_SON:WSON-8-1EP_2x2mm_P0.5mm_EP0.9x1.6mm
- SW1: footprint Button_Switch_SMD:SW_TE_3-1437565-0 -> Button_Switch_SMD:Panasonic_EVQPUL_EVQPUC
- TP1, TP2, TP7: footprint TestPoint:TestPoint_Pad_D0.8mm -> TestPoint:TestPoint_Pad_D1.0mm
- U14: footprint Package_DFN_QFN:VSON-10-1EP_3x3mm_P0.5mm_EP1.7x1.7mm -> Package_SON:VSON-10-1EP_3x3mm_P0.5mm_EP1.65x2.4mm
Changed lines of the file:
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@@
 			)
 		)
-		(property "Footprint" "TestPoint:TestPoint_Pad_D0.8mm"
+		(property "Footprint" "TestPoint:TestPoint_Pad_D1.0mm"
 			(at 160.02 232.2322 0)
 			(hide yes)
@@
 			)
 		)
-		(property "Footprint" "Diode_SMD:D_DFN-2_1x0.6mm_P0.65mm"
+		(property "Footprint" "Package_TO_SOT_SMD:SOT-883"
 			(at 76.2 109.0422 0)
 			(hide yes)
@@
 			)
 		)
-		(property "Footprint" "Package_DFN_QFN:VSON-10-1EP_3x3mm_P0.5mm_EP1.7x1.7mm"
+		(property "Footprint" "Package_SON:VSON-10-1EP_3x3mm_P0.5mm_EP1.65x2.4mm"
 			(at 205.74 226.8982 0)
 			(hide yes)
@@
 			)
 		)
-		(property "Footprint" "Diode_SMD:D_DFN-2_1x0.6mm_P0.65mm"
+		(property "Footprint" "Package_TO_SOT_SMD:SOT-883"
 			(at 66.04 109.0422 0)
 			(hide yes)
@@
 			)
 		)
-		(property "Footprint" "Package_DFN_QFN:VSON-8-1EP_2x2mm_P0.5mm_EP0.9x1.7mm"
+		(property "Footprint" "Package_SON:WSON-8-1EP_2x2mm_P0.5mm_EP0.9x1.6mm"
 			(at 349.25 101.4222 0)
 			(hide yes)
@@
 			)
 		)
-		(property "Footprint" "TestPoint:TestPoint_Pad_D0.8mm"
+		(property "Footprint" "TestPoint:TestPoint_Pad_D1.0mm"
 			(at 124.46 83.6422 0)
 			(hide yes)
@@
 			)
 		)
-		(property "Footprint" "Fiducial:Fiducial_1mm_Silk"
+		(property "Footprint" "Fiducial:Fiducial_1mm_Mask2mm"
 			(at 411.48 215.7222 0)
 			(hide yes)
@@
 			)
 		)
-		(property "Footprint" "Fiducial:Fiducial_1mm_Silk"
+		(property "Footprint" "Fiducial:Fiducial_1mm_Mask2mm"
 			(at 401.32 215.7222 0)
 			(hide yes)
@@
 			)
 		)
-		(property "Footprint" "Fiducial:Fiducial_1mm_Silk"
+		(property "Footprint" "Fiducial:Fiducial_1mm_Mask2mm"
 			(at 391.16 230.9622 0)
 			(hide yes)
@@
 			)
 		)
-		(property "Footprint" "Fiducial:Fiducial_1mm_Silk"
+		(property "Footprint" "Fiducial:Fiducial_1mm_Mask2mm"
 			(at 411.48 230.9622 0)
 			(hide yes)
@@
 			)
 		)
-		(property "Footprint" "TestPoint:TestPoint_Pad_D0.8mm"
+		(property "Footprint" "TestPoint:TestPoint_Pad_D1.0mm"
 			(at 96.52 83.6422 0)
 			(hide yes)
@@
 			)
 		)
-		(property "Footprint" "Button_Switch_SMD:SW_TE_3-1437565-0"
+		(property "Footprint" "Button_Switch_SMD:Panasonic_EVQPUL_EVQPUC"
 			(at 125.73 144.6022 0)
 			(hide yes)
@@
 			)
 		)
-		(property "Footprint" "Fiducial:Fiducial_1mm_Silk"
+		(property "Footprint" "Fiducial:Fiducial_1mm_Mask2mm"
 			(at 401.32 230.9622 0)
 			(hide yes)
@@
 			)
 		)
-		(property "Footprint" "Fiducial:Fiducial_1mm_Silk"
+		(property "Footprint" "Fiducial:Fiducial_1mm_Mask2mm"
 			(at 391.16 215.7222 0)
 			(hide yes)

Commit message: Reset PCB to clean 2-layer layout with fixed enclosure components
- Strip 6-layer Altium PCB down to F.Cu + B.Cu only
- Preserve board outline (149 Edge.Cuts segments)
- Keep 11 mounting holes at original positions
- Lock enclosure-critical components at original positions:
  SW1, U1-U5 (limit sensors, nRF, pressure), J1-J5 (USB-C,
  motor, battery, mic, speaker connectors)
- Preserve BM833 antenna keepout zone
- Fix Altium pin-number artifacts in schematics:
  LED A/K → 1/2, J1 footprint → Amphenol full USB-C,
  Q1 D1/D2/D3/G/S → 5/6/7/8/1, SW1 pins 3/4 → 1/2
- Exclude *.md notes files from git tracking

Co-Authored-By: Claude Sonnet 4.6 <noreply@anthropic.com>
Parts:
- J1: footprint Connector_USB:USB_C_Receptacle_HRO_TYPE-C-31-M-12 -> Connector_USB:USB_C_Receptacle_Amphenol_12401548E4-2A
Connections:
- net GND: now also D12.1 (K), D7.1 (K), J1.SH (SHIELD), Q1.8 (G); no longer D12.K, D7.K, J1.SH1 (SHIELD), J1.SH2 (SHIELD), J1.SH3 (SHIELD), J1.SH4 (SHIELD), Q1.G
- net VBat_IN: now also Q1.5 (D), Q1.6 (D), Q1.7 (D); no longer Q1.D1 (D), Q1.D2 (D), Q1.D3 (D)
- net at C10.2, C9.2, R7.2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: now also Q1.1 (S); no longer Q1.S
- net at R69.1: now also D12.2 (A); no longer D12.A
- net at C44.1, U15.15 (SHPHLD): now also SW1.1 (3), SW1.2 (4); no longer SW1.3, SW1.4
- net at R51.1: now also D7.2 (A); no longer D7.A
Changed lines of the file:
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@@
 			)
 		)
-		(property "Footprint" "Connector_USB:USB_C_Receptacle_HRO_TYPE-C-31-M-12"
+		(property "Footprint" "Connector_USB:USB_C_Receptacle_Amphenol_12401548E4-2A"
 			(at 17.78 109.0422 0)
 			(hide yes)
