File: 065-0200_Main Board (Rev E)/065-0200_Page 3 Micro.kicad_sch (KiCad schematic)
At the start: 36 parts, among them J6 TC2030-CTX, U4 ${PART NUMBER}${DNP}, Y1 ${PART NUMBER}

Commit message: Fix Altium import template variables and footprints in Rev E schematics
- Replace 52 ${PART NUMBER} template variables with actual part numbers
- Replace 180 Altium footprint references with KiCad standard library equivalents
- Placeholders set for BM833, 2SMPP03, custom connectors (need manual assignment)

Co-Authored-By: Claude Sonnet 4.6 <noreply@anthropic.com>
Parts:
- C3, C38, C39, C4, C40, C5, C6, C7, C8: footprint Discretes.PcbLib:CAP_0603 -> Capacitor_SMD:C_0603_1608Metric
- D10, D11, D9: value ${PART NUMBER} -> D5V0H1B2LP-7B; footprint DFN2_1.01X0.61_0.65P -> Diode_SMD:D_DFN-2_1x0.6mm_P0.65mm
- D4, D5, D6: value ${PART NUMBER} -> CLVBA-FKA-CAEDH8BBB7A363; footprint Discretes.PcbLib:LED_PLCC4 - CLVBA -> LED_SMD:LED_PLCC4
- D8: value ${PART NUMBER} -> APT1608ZGCK; footprint Discretes.PcbLib:LED_0603 -> LED_SMD:LED_0603_1608Metric
- J6: footprint TC2030_IDC -> Connector_TagConnect:TC2030-IDC-NL
- R10, R11, R12, R13, R14, R15, R16, R17, R4, R5, R53, R57, R58, R59, R6, R64, R9: footprint Discretes.PcbLib:RES_0603 -> Resistor_SMD:R_0603_1608Metric
- U4: value ${PART NUMBER}${DNP} -> BM833
- Y1: value ${PART NUMBER} -> 9HT10-32.768KBZF-T; footprint Y_2PIN_3.2mmX1.5mm -> Crystal:Crystal_SMD_3215-2Pin_3.2x1.5mm
Changed lines of the file:
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@@
 			)
 		)
-		(property "Footprint" "Discretes.PcbLib:RES_0603"
+		(property "Footprint" "Resistor_SMD:R_0603_1608Metric"
 			(at 406.4 124.2822 0)
 			(hide yes)
@@
 			)
 		)
-		(property "Footprint" "Discretes.PcbLib:RES_0603"
+		(property "Footprint" "Resistor_SMD:R_0603_1608Metric"
 			(at 223.52 73.4822 0)
 			(hide yes)
@@
 			)
 		)
-		(property "Footprint" "Discretes.PcbLib:RES_0603"
+		(property "Footprint" "Resistor_SMD:R_0603_1608Metric"
 			(at 172.72 43.0022 0)
 			(hide yes)
@@
 			)
 		)
-		(property "Footprint" "Discretes.PcbLib:CAP_0603"
+		(property "Footprint" "Capacitor_SMD:C_0603_1608Metric"
 			(at 167.64 45.5422 0)
 			(hide yes)
@@
 			)
 		)
-		(property "Footprint" "Discretes.PcbLib:RES_0603"
+		(property "Footprint" "Resistor_SMD:R_0603_1608Metric"
 			(at 391.16 56.9722 0)
 			(hide yes)
@@
 			)
 		)
-		(property "Footprint" "Discretes.PcbLib:RES_0603"
+		(property "Footprint" "Resistor_SMD:R_0603_1608Metric"
 			(at 83.82 60.7822 0)
 			(hide yes)
@@
 			)
 		)
-		(property "Footprint" "Discretes.PcbLib:CAP_0603"
+		(property "Footprint" "Capacitor_SMD:C_0603_1608Metric"
 			(at 157.48 53.1622 0)
 			(hide yes)
@@
 			)
 		)
-		(property "Footprint" "Discretes.PcbLib:CAP_0603"
+		(property "Footprint" "Capacitor_SMD:C_0603_1608Metric"
 			(at 48.26 93.8022 0)
 			(hide yes)
@@
 			)
 		)
-		(property "Footprint" "Discretes.PcbLib:CAP_0603"
+		(property "Footprint" "Capacitor_SMD:C_0603_1608Metric"
 			(at 106.68 53.1622 0)
 			(hide yes)
@@
 			)
 		)
-		(property "Footprint" "Discretes.PcbLib:RES_0603"
+		(property "Footprint" "Resistor_SMD:R_0603_1608Metric"
 			(at 368.3 56.9722 0)
 			(hide yes)
@@
 			)
 		)
-		(property "Footprint" "Discretes.PcbLib:RES_0603"
+		(property "Footprint" "Resistor_SMD:R_0603_1608Metric"
 			(at 361.95 56.9722 0)
 			(hide yes)
@@
 			)
 		)
-		(property "Footprint" "Discretes.PcbLib:RES_0603"
+		(property "Footprint" "Resistor_SMD:R_0603_1608Metric"
 			(at 397.51 56.9722 0)
 			(hide yes)
@@
 			)
 		)
-		(property "Footprint" "Discretes.PcbLib:RES_0603"
+		(property "Footprint" "Resistor_SMD:R_0603_1608Metric"
 			(at 345.44 56.9722 0)
 			(hide yes)
@@
 			)
 		)
-		(property "Value" "${PART NUMBER}"
+		(property "Value" "D5V0H1B2LP-7B"
 			(at 234.696 257.1242 0)
 			(hide yes)
@@
 			)
 		)
-		(property "Footprint" "DFN2_1.01X0.61_0.65P"
+		(property "Footprint" "Diode_SMD:D_DFN-2_1x0.6mm_P0.65mm"
 			(at 237.49 270.3322 0)
 			(hide yes)
@@
 			)
 		)
-		(property "Value" "${PART NUMBER}"
+		(property "Value" "CLVBA-FKA-CAEDH8BBB7A363"
 			(at 359.156 42.4942 0)
 			(hide yes)
@@
 			)
 		)
-		(property "Footprint" "Discretes.PcbLib:LED_PLCC4 - CLVBA"
+		(property "Footprint" "LED_SMD:LED_PLCC4"
 			(at 368.3 45.5422 0)
 			(hide yes)
@@
 			)
 		)
-		(property "Value" "${PART NUMBER}"
+		(property "Value" "CLVBA-FKA-CAEDH8BBB7A363"
 			(at 336.296 42.4942 0)
 			(hide yes)
@@
 			)
 		)
-		(property "Footprint" "Discretes.PcbLib:LED_PLCC4 - CLVBA"
+		(property "Footprint" "LED_SMD:LED_PLCC4"
 			(at 345.44 45.5422 0)
 			(hide yes)
@@
 			)
 		)
-		(property "Footprint" "Discretes.PcbLib:RES_0603"
+		(property "Footprint" "Resistor_SMD:R_0603_1608Metric"
 			(at 262.89 239.8522 0)
 			(hide yes)
@@
 			)
 		)
-		(property "Value" "${PART NUMBER}"
+		(property "Value" "D5V0H1B2LP-7B"
 			(at 252.476 257.1242 0)
 			(hide yes)
@@
 			)
 		)
-		(property "Footprint" "DFN2_1.01X0.61_0.65P"
+		(property "Footprint" "Diode_SMD:D_DFN-2_1x0.6mm_P0.65mm"
 			(at 255.27 270.3322 0)
 			(hide yes)
@@
 			)
 		)
-		(property "Footprint" "Discretes.PcbLib:RES_0603"
+		(property "Footprint" "Resistor_SMD:R_0603_1608Metric"
 			(at 339.09 56.9722 0)
 			(hide yes)
@@
 			)
 		)
-		(property "Footprint" "Discretes.PcbLib:RES_0603"
+		(property "Footprint" "Resistor_SMD:R_0603_1608Metric"
 			(at 223.52 136.9822 0)
 			(hide yes)
@@
 			)
 		)
-		(property "Footprint" "Discretes.PcbLib:CAP_0603"
+		(property "Footprint" "Capacitor_SMD:C_0603_1608Metric"
 			(at 262.89 265.2522 0)
 			(hide yes)
@@
 			)
 		)
-		(property "Footprint" "TC2030_IDC"
+		(property "Footprint" "Connector_TagConnect:TC2030-IDC-NL"
 			(at 276.86 248.7422 0)
 			(hide yes)
@@
 			)
 		)
-		(property "Value" "${PART NUMBER}"
+		(property "Value" "CLVBA-FKA-CAEDH8BBB7A363"
 			(at 382.016 42.4942 0)
 			(hide yes)
@@
 			)
 		)
-		(property "Footprint" "Discretes.PcbLib:LED_PLCC4 - CLVBA"
+		(property "Footprint" "LED_SMD:LED_PLCC4"
 			(at 391.16 45.5422 0)
 			(hide yes)
@@
 			)
 		)
-		(property "Footprint" "Discretes.PcbLib:RES_0603"
+		(property "Footprint" "Resistor_SMD:R_0603_1608Metric"
 			(at 215.9 73.4822 0)
 			(hide yes)
@@
 			)
 		)
-		(property "Footprint" "Discretes.PcbLib:RES_0603"
+		(property "Footprint" "Resistor_SMD:R_0603_1608Metric"
 			(at 351.79 56.9722 0)
 			(hide yes)
@@
 			)
 		)
-		(property "Value" "${PART NUMBER}${DNP}"
+		(property "Value" "BM833"
 			(at 125.73 67.1322 90)
 			(hide yes)
@@
 			)
 		)
-		(property "Footprint" "Discretes.PcbLib:RES_0603"
+		(property "Footprint" "Resistor_SMD:R_0603_1608Metric"
 			(at 374.65 56.9722 0)
 			(hide yes)
@@
 			)
 		)
-		(property "Value" "${PART NUMBER}"
+		(property "Value" "APT1608ZGCK"
 			(at 403.606 134.9792 0)
 			(hide yes)
@@
 			)
 		)
-		(property "Footprint" "Discretes.PcbLib:LED_0603"
+		(property "Footprint" "LED_SMD:LED_0603_1608Metric"
 			(at 406.4 138.2522 0)
 			(hide yes)
@@
 			)
 		)
-		(property "Value" "${PART NUMBER}"
+		(property "Value" "9HT10-32.768KBZF-T"
 			(at 58.166 94.5642 0)
 			(hide yes)
@@
 			)
 		)
-		(property "Footprint" "Y_2PIN_3.2mmX1.5mm"
+		(property "Footprint" "Crystal:Crystal_SMD_3215-2Pin_3.2x1.5mm"
 			(at 60.96 95.0722 0)
 			(hide yes)
@@
 			)
 		)
-		(property "Footprint" "Discretes.PcbLib:CAP_0603"
+		(property "Footprint" "Capacitor_SMD:C_0603_1608Metric"
 			(at 116.84 45.5422 0)
 			(hide yes)
@@
 			)
 		)
-		(property "Footprint" "Discretes.PcbLib:RES_0603"
+		(property "Footprint" "Resistor_SMD:R_0603_1608Metric"
 			(at 83.82 73.4822 0)
 			(hide yes)
@@
 			)
 		)
-		(property "Footprint" "Discretes.PcbLib:CAP_0603"
+		(property "Footprint" "Capacitor_SMD:C_0603_1608Metric"
 			(at 127 53.1622 0)
 			(hide yes)
@@
 			)
 		)
-		(property "Value" "${PART NUMBER}"
+		(property "Value" "D5V0H1B2LP-7B"
 			(at 243.586 257.1242 0)
 			(hide yes)
@@
 			)
 		)
-		(property "Footprint" "DFN2_1.01X0.61_0.65P"
+		(property "Footprint" "Diode_SMD:D_DFN-2_1x0.6mm_P0.65mm"
 			(at 246.38 270.3322 0)
 			(hide yes)
@@
 			)
 		)
-		(property "Footprint" "Discretes.PcbLib:RES_0603"
+		(property "Footprint" "Resistor_SMD:R_0603_1608Metric"
 			(at 384.81 56.9722 0)
 			(hide yes)
@@
 			)
 		)
-		(property "Footprint" "Discretes.PcbLib:CAP_0603"
+		(property "Footprint" "Capacitor_SMD:C_0603_1608Metric"
 			(at 48.26 109.0422 0)
 			(hide yes)
@@
 			)
 		)
-		(property "Footprint" "Discretes.PcbLib:CAP_0603"
+		(property "Footprint" "Capacitor_SMD:C_0603_1608Metric"
 			(at 96.52 45.5422 0)
 			(hide yes)

Commit message: Fix footprint names to match installed KiCad library
Correct 30 footprint references where library name or footprint name
didn't match KiCad's actual installed libraries (Package_SON vs
Package_DFN_QFN, SOT-363_SC-70-6, Fiducial, SOT-883, etc.)

Co-Authored-By: Claude Sonnet 4.6 <noreply@anthropic.com>
Parts:
- D10, D11, D9: footprint Diode_SMD:D_DFN-2_1x0.6mm_P0.65mm -> Package_TO_SOT_SMD:SOT-883
- D4, D5, D6: footprint LED_SMD:LED_PLCC4 -> LED_SMD:LED_Cree-PLCC4_3.2x2.8mm_CCW
- J6: footprint Connector_TagConnect:TC2030-IDC-NL -> Connector:Tag-Connect_TC2030-IDC-NL_2x03_P1.27mm_Vertical
Changed lines of the file:
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@@
 			)
 		)
-		(property "Footprint" "Diode_SMD:D_DFN-2_1x0.6mm_P0.65mm"
+		(property "Footprint" "Package_TO_SOT_SMD:SOT-883"
 			(at 237.49 270.3322 0)
 			(hide yes)
@@
 			)
 		)
-		(property "Footprint" "LED_SMD:LED_PLCC4"
+		(property "Footprint" "LED_SMD:LED_Cree-PLCC4_3.2x2.8mm_CCW"
 			(at 368.3 45.5422 0)
 			(hide yes)
@@
 			)
 		)
-		(property "Footprint" "LED_SMD:LED_PLCC4"
+		(property "Footprint" "LED_SMD:LED_Cree-PLCC4_3.2x2.8mm_CCW"
 			(at 345.44 45.5422 0)
 			(hide yes)
@@
 			)
 		)
-		(property "Footprint" "Diode_SMD:D_DFN-2_1x0.6mm_P0.65mm"
+		(property "Footprint" "Package_TO_SOT_SMD:SOT-883"
 			(at 255.27 270.3322 0)
 			(hide yes)
@@
 			)
 		)
-		(property "Footprint" "Connector_TagConnect:TC2030-IDC-NL"
+		(property "Footprint" "Connector:Tag-Connect_TC2030-IDC-NL_2x03_P1.27mm_Vertical"
 			(at 276.86 248.7422 0)
 			(hide yes)
@@
 			)
 		)
-		(property "Footprint" "LED_SMD:LED_PLCC4"
+		(property "Footprint" "LED_SMD:LED_Cree-PLCC4_3.2x2.8mm_CCW"
 			(at 391.16 45.5422 0)
 			(hide yes)
@@
 			)
 		)
-		(property "Footprint" "Diode_SMD:D_DFN-2_1x0.6mm_P0.65mm"
+		(property "Footprint" "Package_TO_SOT_SMD:SOT-883"
 			(at 246.38 270.3322 0)
 			(hide yes)

Commit message: Reset PCB to clean 2-layer layout with fixed enclosure components
- Strip 6-layer Altium PCB down to F.Cu + B.Cu only
- Preserve board outline (149 Edge.Cuts segments)
- Keep 11 mounting holes at original positions
- Lock enclosure-critical components at original positions:
  SW1, U1-U5 (limit sensors, nRF, pressure), J1-J5 (USB-C,
  motor, battery, mic, speaker connectors)
- Preserve BM833 antenna keepout zone
- Fix Altium pin-number artifacts in schematics:
  LED A/K → 1/2, J1 footprint → Amphenol full USB-C,
  Q1 D1/D2/D3/G/S → 5/6/7/8/1, SW1 pins 3/4 → 1/2
- Exclude *.md notes files from git tracking

Co-Authored-By: Claude Sonnet 4.6 <noreply@anthropic.com>
Connections:
- net HEARTBEAT: now also D8.1 (K); no longer D8.K
- net at R53.1: now also D8.2 (A); no longer D8.A

Commit message: Add OLED display connector to Micro schematic
Added J7 (GME12864-13 OLED) 4-pin I2C connector on Page 3 Micro,
wired to existing SDA/SCL nets shared with the nRF module.

Co-Authored-By: Claude Sonnet 4.6 <noreply@anthropic.com>
Parts:
- added J7: Conn_01x04_Pin, Connector_PinHeader_2.54mm:PinHeader_1x04_P2.54mm_Vertical, symbol Connector:Conn_01x04_Pin
Connections:
- net +3V3: now also J7.3 (Pin_3)
- net GND: now also J7.4 (Pin_4)
- net SCL: now also J7.2 (Pin_2)
- net SDA: now also J7.1 (Pin_1)
Other:
- note added: "OLED Screen"
