File: 065-0200_Main Board (Rev E)/065-0200_Page 4 Sensors.kicad_sch (KiCad schematic)
At the start: 38 parts, among them J4 custom_3p_2mm, U12 LM393DMR2G, U13 ${PART NUMBER}, U5 ${PART NUMBER}, U6 ${PART NUMBER}, U7 INA326, U9 ${PART NUMBER}

Commit message: Fix Altium import template variables and footprints in Rev E schematics
- Replace 52 ${PART NUMBER} template variables with actual part numbers
- Replace 180 Altium footprint references with KiCad standard library equivalents
- Placeholders set for BM833, 2SMPP03, custom connectors (need manual assignment)

Co-Authored-By: Claude Sonnet 4.6 <noreply@anthropic.com>
Parts:
- C14, C15, C17, C18, C19, C20, C22, C23, C26, C27, C29, C32: footprint Discretes.PcbLib:CAP_0603 -> Capacitor_SMD:C_0603_1608Metric
- J4: footprint Connectors.PcbLib:Custom_3p-2MM -> Connector_PinHeader_2.00mm:PinHeader_1x03_P2.00mm_Vertical
- R18, R19, R22, R25, R26, R27, R29, R30, R31, R32, R33, R35, R38, R39, R43, R44: footprint Discretes.PcbLib:RES_0603 -> Resistor_SMD:R_0603_1608Metric
- R28: value ${PART NUMBER} -> ERJ-3EKF6810V; footprint Discretes.PcbLib:RES_0603 -> Resistor_SMD:R_0603_1608Metric
- R36: footprint Discretes.PcbLib:RES_0805 -> Resistor_SMD:R_0805_2012Metric
- TP3: footprint TP_TH_45-25 -> TestPoint:TestPoint_THTPad_D1.143mm_Drill0.635mm
- U12: footprint IC packages.PcbLib:MICRO8 3.3X3.3.1 -> Package_SO:SOIC-8_3.9x4.9mm_P1.27mm
- U12: value ${PARTNUMBER} -> LM393DMR2G; footprint IC packages.PcbLib:MICRO8 3.3X3.3.1 -> Package_SO:SOIC-8_3.9x4.9mm_P1.27mm
- U13: value ${PART NUMBER} -> MAX9109EUT+T; footprint SOT23-6 -> Package_TO_SOT_SMD:SOT-23-6; PACKAGEDESCRIPTION SOT23-6 -> Package_TO_SOT_SMD:SOT-23-6; PACKAGEREFERENCE SOT23-6 -> Package_TO_SOT_SMD:SOT-23-6
- U5: value ${PART NUMBER} -> 2SMPP03; footprint 6SOP_2SMPP-03 -> Package_SO:SOIC-6_3.9x4.9mm_P1.27mm
- U6: value ${PART NUMBER} -> TLV313IDBVT; footprint IC packages.PcbLib:SOT-23-5 -> Package_TO_SOT_SMD:SOT-23-5
- U7: footprint TSSOP-8_3x3 -> Package_SO:TSSOP-8_3x3mm_P0.65mm
- U9: value ${PART NUMBER} -> LM334MX/NOPB; footprint 8-SOIC -> Package_SO:SOIC-8_3.9x4.9mm_P1.27mm; PACKAGEREFERENCE 8-SOIC -> Package_SO:SOIC-8_3.9x4.9mm_P1.27mm
Changed lines of the file:
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@@
 			)
 		)
-		(property "Footprint" "Discretes.PcbLib:CAP_0603"
+		(property "Footprint" "Capacitor_SMD:C_0603_1608Metric"
 			(at 104.14 215.7222 0)
 			(hide yes)
@@
 			)
 		)
-		(property "Footprint" "TP_TH_45-25"
+		(property "Footprint" "TestPoint:TestPoint_THTPad_D1.143mm_Drill0.635mm"
 			(at 213.36 208.1022 0)
 			(hide yes)
@@
 			)
 		)
-		(property "Footprint" "Discretes.PcbLib:CAP_0603"
+		(property "Footprint" "Capacitor_SMD:C_0603_1608Metric"
 			(at 210.82 76.0222 0)
 			(hide yes)
@@
 			)
 		)
-		(property "Footprint" "Discretes.PcbLib:RES_0603"
+		(property "Footprint" "Resistor_SMD:R_0603_1608Metric"
 			(at 335.28 63.3222 0)
 			(hide yes)
@@
 			)
 		)
-		(property "Footprint" "Discretes.PcbLib:RES_0603"
+		(property "Footprint" "Resistor_SMD:R_0603_1608Metric"
 			(at 139.7 214.4522 0)
 			(hide yes)
@@
 			)
 		)
-		(property "Footprint" "TSSOP-8_3x3"
+		(property "Footprint" "Package_SO:TSSOP-8_3x3mm_P0.65mm"
 			(at 170.18 73.4822 0)
 			(hide yes)
@@
 			)
 		)
-		(property "Footprint" "Discretes.PcbLib:RES_0603"
+		(property "Footprint" "Resistor_SMD:R_0603_1608Metric"
 			(at 358.14 45.5422 0)
 			(hide yes)
@@
 			)
 		)
-		(property "Footprint" "Discretes.PcbLib:CAP_0603"
+		(property "Footprint" "Capacitor_SMD:C_0603_1608Metric"
 			(at 205.74 95.0722 0)
 			(hide yes)
@@
 			)
 		)
-		(property "Footprint" "Discretes.PcbLib:RES_0603"
+		(property "Footprint" "Resistor_SMD:R_0603_1608Metric"
 			(at 200.66 220.8022 0)
 			(hide yes)
@@
 			)
 		)
-		(property "Footprint" "Discretes.PcbLib:CAP_0603"
+		(property "Footprint" "Capacitor_SMD:C_0603_1608Metric"
 			(at 180.34 63.3222 0)
 			(hide yes)
@@
 			)
 		)
-		(property "Value" "${PART NUMBER}"
+		(property "Value" "LM334MX/NOPB"
 			(at 84.328 53.1622 90)
 			(show_name no)
@@
 			)
 		)
-		(property "Footprint" "8-SOIC"
+		(property "Footprint" "Package_SO:SOIC-8_3.9x4.9mm_P1.27mm"
 			(at 66.04 50.6222 0)
 			(hide yes)
@@
 			)
 		)
-		(property "PACKAGEREFERENCE" "8-SOIC"
+		(property "PACKAGEREFERENCE" "Package_SO:SOIC-8_3.9x4.9mm_P1.27mm"
 			(at 60.452 46.8122 90)
 			(hide yes)
@@
 			)
 		)
-		(property "Footprint" "Discretes.PcbLib:RES_0603"
+		(property "Footprint" "Resistor_SMD:R_0603_1608Metric"
 			(at 195.58 93.8022 0)
 			(hide yes)
@@
 			)
 		)
-		(property "Footprint" "Discretes.PcbLib:CAP_0603"
+		(property "Footprint" "Capacitor_SMD:C_0603_1608Metric"
 			(at 391.16 53.1622 0)
 			(hide yes)
@@
 			)
 		)
-		(property "Footprint" "Discretes.PcbLib:CAP_0603"
+		(property "Footprint" "Capacitor_SMD:C_0603_1608Metric"
 			(at 132.08 214.4522 0)
 			(hide yes)
@@
 			)
 		)
-		(property "Footprint" "Discretes.PcbLib:RES_0603"
+		(property "Footprint" "Resistor_SMD:R_0603_1608Metric"
 			(at 91.44 205.5622 0)
 			(hide yes)
@@
 			)
 		)
-		(property "Footprint" "Discretes.PcbLib:RES_0805"
+		(property "Footprint" "Resistor_SMD:R_0805_2012Metric"
 			(at 73.66 203.0222 0)
 			(hide yes)
@@
 			)
 		)
-		(property "Footprint" "Discretes.PcbLib:CAP_0603"
+		(property "Footprint" "Capacitor_SMD:C_0603_1608Metric"
 			(at 187.96 185.2422 0)
 			(hide yes)
@@
 			)
 		)
-		(property "Footprint" "Discretes.PcbLib:RES_0603"
+		(property "Footprint" "Resistor_SMD:R_0603_1608Metric"
 			(at 121.92 196.6722 0)
 			(hide yes)
@@
 			)
 		)
-		(property "Footprint" "Discretes.PcbLib:RES_0603"
+		(property "Footprint" "Resistor_SMD:R_0603_1608Metric"
 			(at 152.4 68.4022 0)
 			(hide yes)
@@
 			)
 		)
-		(property "Footprint" "Discretes.PcbLib:RES_0603"
+		(property "Footprint" "Resistor_SMD:R_0603_1608Metric"
 			(at 264.16 53.1622 0)
 			(hide yes)
@@
 			)
 		)
-		(property "Footprint" "Discretes.PcbLib:CAP_0603"
+		(property "Footprint" "Capacitor_SMD:C_0603_1608Metric"
 			(at 139.7 204.2922 0)
 			(hide yes)
@@
 			)
 		)
-		(property "Value" "${PART NUMBER}"
+		(property "Value" "TLV313IDBVT"
 			(at 193.548 200.2282 90)
 			(show_name no)
@@
 			)
 		)
-		(property "Footprint" "IC packages.PcbLib:SOT-23-5"
+		(property "Footprint" "Package_TO_SOT_SMD:SOT-23-5"
 			(at 172.72 200.4822 0)
 			(hide yes)
@@
 			)
 		)
-		(property "Footprint" "Discretes.PcbLib:RES_0603"
+		(property "Footprint" "Resistor_SMD:R_0603_1608Metric"
 			(at 96.52 68.4022 0)
 			(hide yes)
@@
 			)
 		)
-		(property "Footprint" "Discretes.PcbLib:CAP_0603"
+		(property "Footprint" "Capacitor_SMD:C_0603_1608Metric"
 			(at 314.96 65.8622 0)
 			(hide yes)
@@
 			)
 		)
-		(property "Footprint" "Discretes.PcbLib:RES_0603"
+		(property "Footprint" "Resistor_SMD:R_0603_1608Metric"
 			(at 198.12 73.4822 0)
 			(hide yes)
@@
 			)
 		)
-		(property "Footprint" "Connectors.PcbLib:Custom_3p-2MM"
+		(property "Footprint" "Connector_PinHeader_2.00mm:PinHeader_1x03_P2.00mm_Vertical"
 			(at 71.12 208.1022 0)
 			(hide yes)
@@
 			)
 		)
-		(property "Footprint" "Discretes.PcbLib:RES_0603"
+		(property "Footprint" "Resistor_SMD:R_0603_1608Metric"
 			(at 264.16 83.6422 0)
 			(hide yes)
@@
 			)
 		)
-		(property "Footprint" "Discretes.PcbLib:RES_0603"
+		(property "Footprint" "Resistor_SMD:R_0603_1608Metric"
 			(at 195.58 81.1022 0)
 			(hide yes)
@@
 			)
 		)
-		(property "Footprint" "IC packages.PcbLib:MICRO8 3.3X3.3.1"
+		(property "Footprint" "Package_SO:SOIC-8_3.9x4.9mm_P1.27mm"
 			(at 302.26 63.3222 0)
 			(hide yes)
@@
 			)
 		)
-		(property "Footprint" "Discretes.PcbLib:RES_0603"
+		(property "Footprint" "Resistor_SMD:R_0603_1608Metric"
 			(at 167.64 220.8022 0)
 			(hide yes)
@@
 			)
 		)
-		(property "Value" "${PART NUMBER}"
+		(property "Value" "ERJ-3EKF6810V"
 			(at 86.106 64.0842 90)
 			(hide yes)
@@
 			)
 		)
-		(property "Footprint" "Discretes.PcbLib:RES_0603"
+		(property "Footprint" "Resistor_SMD:R_0603_1608Metric"
 			(at 86.36 58.2422 0)
 			(hide yes)
@@
 			)
 		)
-		(property "Footprint" "Discretes.PcbLib:RES_0603"
+		(property "Footprint" "Resistor_SMD:R_0603_1608Metric"
 			(at 358.14 55.7022 0)
 			(hide yes)
@@
 			)
 		)
-		(property "Footprint" "Discretes.PcbLib:CAP_0603"
+		(property "Footprint" "Capacitor_SMD:C_0603_1608Metric"
 			(at 71.12 180.1622 0)
 			(hide yes)
@@
 			)
 		)
-		(property "Value" "${PART NUMBER}"
+		(property "Value" "2SMPP03"
 			(at 114.3 83.6422 90)
 			(show_name no)
@@
 			)
 		)
-		(property "Footprint" "6SOP_2SMPP-03"
+		(property "Footprint" "Package_SO:SOIC-6_3.9x4.9mm_P1.27mm"
 			(at 114.3 65.8622 0)
 			(hide yes)
@@
 			)
 		)
-		(property "Footprint" "Discretes.PcbLib:CAP_0603"
+		(property "Footprint" "Capacitor_SMD:C_0603_1608Metric"
 			(at 60.96 172.5422 0)
 			(hide yes)
@@
 			)
 		)
-		(property "Footprint" "Discretes.PcbLib:CAP_0603"
+		(property "Footprint" "Capacitor_SMD:C_0603_1608Metric"
 			(at 55.88 50.6222 0)
 			(hide yes)
@@
 			)
 		)
-		(property "Footprint" "Discretes.PcbLib:RES_0603"
+		(property "Footprint" "Resistor_SMD:R_0603_1608Metric"
 			(at 264.16 68.4022 0)
 			(hide yes)
@@
 			)
 		)
-		(property "Value" "${PARTNUMBER}"
+		(property "Value" "LM393DMR2G"
 			(at 314.96 93.8022 90)
 			(show_name no)
@@
 			)
 		)
-		(property "Footprint" "IC packages.PcbLib:MICRO8 3.3X3.3.1"
+		(property "Footprint" "Package_SO:SOIC-8_3.9x4.9mm_P1.27mm"
 			(at 302.26 92.5322 0)
 			(hide yes)
@@
 			)
 		)
-		(property "Value" "${PART NUMBER}"
+		(property "Value" "MAX9109EUT+T"
 			(at 387.35 88.7222 90)
 			(show_name no)
@@
 			)
 		)
-		(property "Footprint" "SOT23-6"
+		(property "Footprint" "Package_TO_SOT_SMD:SOT-23-6"
 			(at 370.84 68.4022 0)
 			(hide yes)
@@
 			)
 		)
-		(property "PACKAGEREFERENCE" "SOT23-6"
+		(property "PACKAGEREFERENCE" "Package_TO_SOT_SMD:SOT-23-6"
 			(at 370.84 68.4022 90)
 			(hide yes)
@@
 			)
 		)
-		(property "PACKAGEDESCRIPTION" "SOT23-6"
+		(property "PACKAGEDESCRIPTION" "Package_TO_SOT_SMD:SOT-23-6"
 			(at 370.84 68.4022 90)
 			(hide yes)

Commit message: Fix footprint names to match installed KiCad library
Correct 30 footprint references where library name or footprint name
didn't match KiCad's actual installed libraries (Package_SON vs
Package_DFN_QFN, SOT-363_SC-70-6, Fiducial, SOT-883, etc.)

Co-Authored-By: Claude Sonnet 4.6 <noreply@anthropic.com>
Parts:
- TP3: footprint TestPoint:TestPoint_THTPad_D1.143mm_Drill0.635mm -> TestPoint:TestPoint_THTPad_D1.5mm_Drill0.7mm
- U5: footprint Package_SO:SOIC-6_3.9x4.9mm_P1.27mm -> Package_SO:SOIC-8_3.9x4.9mm_P1.27mm
Changed lines of the file:
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@@
 			)
 		)
-		(property "Footprint" "TestPoint:TestPoint_THTPad_D1.143mm_Drill0.635mm"
+		(property "Footprint" "TestPoint:TestPoint_THTPad_D1.5mm_Drill0.7mm"
 			(at 213.36 208.1022 0)
 			(hide yes)
@@
 			)
 		)
-		(property "Footprint" "Package_SO:SOIC-6_3.9x4.9mm_P1.27mm"
+		(property "Footprint" "Package_SO:SOIC-8_3.9x4.9mm_P1.27mm"
 			(at 114.3 65.8622 0)
 			(hide yes)
