File: 065-0200_Main Board (Rev E)/065-0200_Page 5 Motor Driver.kicad_sch (KiCad schematic)
At the start: 17 parts, among them J2 ${PART NUMBER}, U1 QRE1113GR, U16 ${PART NUMBER}, U2 QRE1113GR, U3 QRE1113GR, U8 ${PART NUMBER}

Commit message: Fix Altium import template variables and footprints in Rev E schematics
- Replace 52 ${PART NUMBER} template variables with actual part numbers
- Replace 180 Altium footprint references with KiCad standard library equivalents
- Placeholders set for BM833, 2SMPP03, custom connectors (need manual assignment)

Co-Authored-By: Claude Sonnet 4.6 <noreply@anthropic.com>
Parts:
- C41, C42, C43: footprint Discretes.PcbLib:CAP_0603 -> Capacitor_SMD:C_0603_1608Metric
- J2: value ${PART NUMBER} -> 0022035025; footprint Molex_2P-2.50_22035025 -> Connector_PinHeader_2.54mm:PinHeader_1x02_P2.54mm_Vertical
- R60, R61, R62, R63, R65, R66, R67, R68: footprint Discretes.PcbLib:RES_0603 -> Resistor_SMD:R_0603_1608Metric
- U1, U2, U3: footprint SOIC180P460X187-4N -> Sensor_Optical:QRE1113_SMD
- U16: value ${PART NUMBER} -> 74LVC1G27GW,12; footprint SOT_363 -> Package_TO_SOT_SMD:SOT-363
- U8: value ${PART NUMBER} -> DRV8837DSGR; footprint WSON_8_2X2 -> Package_DFN_QFN:WSON-8-1EP_2x2mm_P0.5mm_EP0.9x1.6mm
Changed lines of the file:
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@@
 			)
 		)
-		(property "Footprint" "Discretes.PcbLib:RES_0603"
+		(property "Footprint" "Resistor_SMD:R_0603_1608Metric"
 			(at 350.52 175.0822 0)
 			(hide yes)
@@
 			)
 		)
-		(property "Footprint" "Discretes.PcbLib:RES_0603"
+		(property "Footprint" "Resistor_SMD:R_0603_1608Metric"
 			(at 350.52 98.8822 0)
 			(hide yes)
@@
 			)
 		)
-		(property "Footprint" "Discretes.PcbLib:RES_0603"
+		(property "Footprint" "Resistor_SMD:R_0603_1608Metric"
 			(at 317.5 109.0422 0)
 			(hide yes)
@@
 			)
 		)
-		(property "Footprint" "SOIC180P460X187-4N"
+		(property "Footprint" "Sensor_Optical:QRE1113_SMD"
 			(at 330.2 106.5022 0)
 			(hide yes)
@@
 			)
 		)
-		(property "Footprint" "Discretes.PcbLib:CAP_0603"
+		(property "Footprint" "Capacitor_SMD:C_0603_1608Metric"
 			(at 157.48 76.0222 0)
 			(hide yes)
@@
 			)
 		)
-		(property "Footprint" "SOIC180P460X187-4N"
+		(property "Footprint" "Sensor_Optical:QRE1113_SMD"
 			(at 330.2 144.6022 0)
 			(hide yes)
@@
 			)
 		)
-		(property "Footprint" "Discretes.PcbLib:RES_0603"
+		(property "Footprint" "Resistor_SMD:R_0603_1608Metric"
 			(at 114.3 119.2022 0)
 			(hide yes)
@@
 			)
 		)
-		(property "Footprint" "Discretes.PcbLib:RES_0603"
+		(property "Footprint" "Resistor_SMD:R_0603_1608Metric"
 			(at 350.52 136.9822 0)
 			(hide yes)
@@
 			)
 		)
-		(property "Footprint" "Discretes.PcbLib:RES_0603"
+		(property "Footprint" "Resistor_SMD:R_0603_1608Metric"
 			(at 106.68 119.2022 0)
 			(hide yes)
@@
 			)
 		)
-		(property "Value" "${PART NUMBER}"
+		(property "Value" "DRV8837DSGR"
 			(at 157.988 96.3422 90)
 			(show_name no)
@@
 			)
 		)
-		(property "Footprint" "WSON_8_2X2"
+		(property "Footprint" "Package_DFN_QFN:WSON-8-1EP_2x2mm_P0.5mm_EP0.9x1.6mm"
 			(at 121.92 96.3422 0)
 			(hide yes)
@@
 			)
 		)
-		(property "Footprint" "Discretes.PcbLib:RES_0603"
+		(property "Footprint" "Resistor_SMD:R_0603_1608Metric"
 			(at 317.5 147.1422 0)
 			(hide yes)
@@
 			)
 		)
-		(property "Footprint" "SOIC180P460X187-4N"
+		(property "Footprint" "Sensor_Optical:QRE1113_SMD"
 			(at 330.2 182.7022 0)
 			(hide yes)
@@
 			)
 		)
-		(property "Footprint" "Discretes.PcbLib:CAP_0603"
+		(property "Footprint" "Capacitor_SMD:C_0603_1608Metric"
 			(at 63.5 93.8022 0)
 			(hide yes)
@@
 			)
 		)
-		(property "Value" "${PART NUMBER}"
+		(property "Value" "74LVC1G27GW,12"
 			(at 70.612 114.8842 90)
 			(show_name no)
@@
 			)
 		)
-		(property "Footprint" "SOT_363"
+		(property "Footprint" "Package_TO_SOT_SMD:SOT-363"
 			(at 63.5 111.5822 0)
 			(hide yes)
@@
 			)
 		)
-		(property "Value" "${PART NUMBER}"
+		(property "Value" "0022035025"
 			(at 187.96 124.2822 90)
 			(hide yes)
@@
 			)
 		)
-		(property "Footprint" "Molex_2P-2.50_22035025"
+		(property "Footprint" "Connector_PinHeader_2.54mm:PinHeader_1x02_P2.54mm_Vertical"
 			(at 187.96 103.9622 0)
 			(hide yes)
@@
 			)
 		)
-		(property "Footprint" "Discretes.PcbLib:CAP_0603"
+		(property "Footprint" "Capacitor_SMD:C_0603_1608Metric"
 			(at 121.92 76.0222 0)
 			(hide yes)
@@
 			)
 		)
-		(property "Footprint" "Discretes.PcbLib:RES_0603"
+		(property "Footprint" "Resistor_SMD:R_0603_1608Metric"
 			(at 317.5 185.2422 0)
 			(hide yes)

Commit message: Fix footprint names to match installed KiCad library
Correct 30 footprint references where library name or footprint name
didn't match KiCad's actual installed libraries (Package_SON vs
Package_DFN_QFN, SOT-363_SC-70-6, Fiducial, SOT-883, etc.)

Co-Authored-By: Claude Sonnet 4.6 <noreply@anthropic.com>
Parts:
- U1, U2, U3: footprint Sensor_Optical:QRE1113_SMD -> Package_SO:SOIC-4_4.55x2.6mm_P1.27mm
- U16: footprint Package_TO_SOT_SMD:SOT-363 -> Package_TO_SOT_SMD:SOT-363_SC-70-6
- U8: footprint Package_DFN_QFN:WSON-8-1EP_2x2mm_P0.5mm_EP0.9x1.6mm -> Package_SON:WSON-8-1EP_2x2mm_P0.5mm_EP0.9x1.6mm
Changed lines of the file:
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@@
 			)
 		)
-		(property "Footprint" "Sensor_Optical:QRE1113_SMD"
+		(property "Footprint" "Package_SO:SOIC-4_4.55x2.6mm_P1.27mm"
 			(at 330.2 106.5022 0)
 			(hide yes)
@@
 			)
 		)
-		(property "Footprint" "Sensor_Optical:QRE1113_SMD"
+		(property "Footprint" "Package_SO:SOIC-4_4.55x2.6mm_P1.27mm"
 			(at 330.2 144.6022 0)
 			(hide yes)
@@
 			)
 		)
-		(property "Footprint" "Package_DFN_QFN:WSON-8-1EP_2x2mm_P0.5mm_EP0.9x1.6mm"
+		(property "Footprint" "Package_SON:WSON-8-1EP_2x2mm_P0.5mm_EP0.9x1.6mm"
 			(at 121.92 96.3422 0)
 			(hide yes)
@@
 			)
 		)
-		(property "Footprint" "Sensor_Optical:QRE1113_SMD"
+		(property "Footprint" "Package_SO:SOIC-4_4.55x2.6mm_P1.27mm"
 			(at 330.2 182.7022 0)
 			(hide yes)
@@
 			)
 		)
-		(property "Footprint" "Package_TO_SOT_SMD:SOT-363"
+		(property "Footprint" "Package_TO_SOT_SMD:SOT-363_SC-70-6"
 			(at 63.5 111.5822 0)
 			(hide yes)
