File: 065-0200_Main Board (Rev E)/065-0200_Page 6 Audio.kicad_sch (KiCad schematic)
At the start: 21 parts, among them J5 custom_2p_2mm, U10 ${PART NUMBER}, U11 ${PART NUMBER}

Commit message: Fix Altium import template variables and footprints in Rev E schematics
- Replace 52 ${PART NUMBER} template variables with actual part numbers
- Replace 180 Altium footprint references with KiCad standard library equivalents
- Placeholders set for BM833, 2SMPP03, custom connectors (need manual assignment)

Co-Authored-By: Claude Sonnet 4.6 <noreply@anthropic.com>
Parts:
- C11, C12, C13, C16, C21, C24, C25, C28: footprint Discretes.PcbLib:CAP_0603 -> Capacitor_SMD:C_0603_1608Metric
- J5: footprint Custom_2p-2MM -> Connector_PinHeader_2.00mm:PinHeader_1x02_P2.00mm_Vertical
- R20, R21, R23, R24, R37, R70, R71: footprint Discretes.PcbLib:RES_0603 -> Resistor_SMD:R_0603_1608Metric
- R34: footprint Discretes.PcbLib:RES_0805 -> Resistor_SMD:R_0805_2012Metric
- TP4, TP5: footprint TP_TH_45-25 -> TestPoint:TestPoint_THTPad_D1.143mm_Drill0.635mm
- U10: value ${PART NUMBER} -> LM4875MM/NOPB; footprint MSOP-8_MPS -> Package_SO:MSOP-8_3x3mm_P0.65mm
- U11: value ${PART NUMBER} -> TLV313IDBVT; footprint IC packages.PcbLib:SOT-23-5 -> Package_TO_SOT_SMD:SOT-23-5
Changed lines of the file:
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@@
 			)
 		)
-		(property "Footprint" "Discretes.PcbLib:RES_0603"
+		(property "Footprint" "Resistor_SMD:R_0603_1608Metric"
 			(at 185.42 116.6622 0)
 			(hide yes)
@@
 			)
 		)
-		(property "Footprint" "Discretes.PcbLib:CAP_0603"
+		(property "Footprint" "Capacitor_SMD:C_0603_1608Metric"
 			(at 116.84 98.8822 0)
 			(hide yes)
@@
 			)
 		)
-		(property "Footprint" "Discretes.PcbLib:RES_0603"
+		(property "Footprint" "Resistor_SMD:R_0603_1608Metric"
 			(at 97.79 91.2622 0)
 			(hide yes)
@@
 			)
 		)
-		(property "Footprint" "Discretes.PcbLib:RES_0603"
+		(property "Footprint" "Resistor_SMD:R_0603_1608Metric"
 			(at 97.79 119.2022 0)
 			(hide yes)
@@
 			)
 		)
-		(property "Footprint" "Discretes.PcbLib:CAP_0603"
+		(property "Footprint" "Capacitor_SMD:C_0603_1608Metric"
 			(at 226.06 73.4822 0)
 			(hide yes)
@@
 			)
 		)
-		(property "Footprint" "Discretes.PcbLib:CAP_0603"
+		(property "Footprint" "Capacitor_SMD:C_0603_1608Metric"
 			(at 129.54 76.0222 0)
 			(hide yes)
@@
 			)
 		)
-		(property "Footprint" "Discretes.PcbLib:RES_0603"
+		(property "Footprint" "Resistor_SMD:R_0603_1608Metric"
 			(at 127 119.2022 0)
 			(hide yes)
@@
 			)
 		)
-		(property "Value" "${PART NUMBER}"
+		(property "Value" "LM4875MM/NOPB"
 			(at 234.188 93.8022 90)
 			(show_name no)
@@
 			)
 		)
-		(property "Footprint" "MSOP-8_MPS"
+		(property "Footprint" "Package_SO:MSOP-8_3x3mm_P0.65mm"
 			(at 203.2 93.8022 0)
 			(hide yes)
@@
 			)
 		)
-		(property "Footprint" "Discretes.PcbLib:RES_0603"
+		(property "Footprint" "Resistor_SMD:R_0603_1608Metric"
 			(at 116.84 119.2022 0)
 			(hide yes)
@@
 			)
 		)
-		(property "Footprint" "Discretes.PcbLib:RES_0603"
+		(property "Footprint" "Resistor_SMD:R_0603_1608Metric"
 			(at 165.1 119.2022 0)
 			(hide yes)
@@
 			)
 		)
-		(property "Footprint" "Custom_2p-2MM"
+		(property "Footprint" "Connector_PinHeader_2.00mm:PinHeader_1x02_P2.00mm_Vertical"
 			(at 274.32 93.8022 0)
 			(hide yes)
@@
 			)
 		)
-		(property "Footprint" "TP_TH_45-25"
+		(property "Footprint" "TestPoint:TestPoint_THTPad_D1.143mm_Drill0.635mm"
 			(at 261.62 95.0722 0)
 			(hide yes)
@@
 			)
 		)
-		(property "Footprint" "Discretes.PcbLib:CAP_0603"
+		(property "Footprint" "Capacitor_SMD:C_0603_1608Metric"
 			(at 142.24 126.8222 0)
 			(hide yes)
@@
 			)
 		)
-		(property "Footprint" "Discretes.PcbLib:CAP_0603"
+		(property "Footprint" "Capacitor_SMD:C_0603_1608Metric"
 			(at 151.13 126.8222 0)
 			(hide yes)
@@
 			)
 		)
-		(property "Footprint" "Discretes.PcbLib:CAP_0603"
+		(property "Footprint" "Capacitor_SMD:C_0603_1608Metric"
 			(at 238.76 109.0422 0)
 			(hide yes)
@@
 			)
 		)
-		(property "Footprint" "TP_TH_45-25"
+		(property "Footprint" "TestPoint:TestPoint_THTPad_D1.143mm_Drill0.635mm"
 			(at 261.62 98.8822 0)
 			(hide yes)
@@
 			)
 		)
-		(property "Value" "${PART NUMBER}"
+		(property "Value" "TLV313IDBVT"
 			(at 152.908 91.0082 90)
 			(show_name no)
@@
 			)
 		)
-		(property "Footprint" "IC packages.PcbLib:SOT-23-5"
+		(property "Footprint" "Package_TO_SOT_SMD:SOT-23-5"
 			(at 132.08 91.2622 0)
 			(hide yes)
@@
 			)
 		)
-		(property "Footprint" "Discretes.PcbLib:CAP_0603"
+		(property "Footprint" "Capacitor_SMD:C_0603_1608Metric"
 			(at 160.02 126.8222 0)
 			(hide yes)
@@
 			)
 		)
-		(property "Footprint" "Discretes.PcbLib:RES_0805"
+		(property "Footprint" "Resistor_SMD:R_0805_2012Metric"
 			(at 238.76 100.1522 0)
 			(hide yes)
@@
 			)
 		)
-		(property "Footprint" "Discretes.PcbLib:CAP_0603"
+		(property "Footprint" "Capacitor_SMD:C_0603_1608Metric"
 			(at 170.18 93.8022 0)
 			(hide yes)
@@
 			)
 		)
-		(property "Footprint" "Discretes.PcbLib:RES_0603"
+		(property "Footprint" "Resistor_SMD:R_0603_1608Metric"
 			(at 185.42 106.5022 0)
 			(hide yes)

Commit message: Fix footprint names to match installed KiCad library
Correct 30 footprint references where library name or footprint name
didn't match KiCad's actual installed libraries (Package_SON vs
Package_DFN_QFN, SOT-363_SC-70-6, Fiducial, SOT-883, etc.)

Co-Authored-By: Claude Sonnet 4.6 <noreply@anthropic.com>
Parts:
- TP4, TP5: footprint TestPoint:TestPoint_THTPad_D1.143mm_Drill0.635mm -> TestPoint:TestPoint_THTPad_D1.5mm_Drill0.7mm
Changed lines of the file:
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@@
 			)
 		)
-		(property "Footprint" "TestPoint:TestPoint_THTPad_D1.143mm_Drill0.635mm"
+		(property "Footprint" "TestPoint:TestPoint_THTPad_D1.5mm_Drill0.7mm"
 			(at 261.62 95.0722 0)
 			(hide yes)
@@
 			)
 		)
-		(property "Footprint" "TestPoint:TestPoint_THTPad_D1.143mm_Drill0.635mm"
+		(property "Footprint" "TestPoint:TestPoint_THTPad_D1.5mm_Drill0.7mm"
 			(at 261.62 98.8822 0)
 			(hide yes)
